File: GTC_SYSTEM_01.sch (KiCad schematic (older format))
At the start: 11 parts

Commit message: GTC_SYSTEM_01 schem upate
Connections:
- net at CONTROL?.GND: now also PS?.2 (GND)
- net at CONTROL?.VIN (12-24VDC): now also PS?.1 (+24VDC)
Other:
- note added: "DIN\nRAIL"
- note added: "HEATER DRIVER OUTPUT MODULE"
- note added: "Lower Deck Screw Terminals"
- note added: "RTD TEMPERATURE SENSOR MODULE"
- note added: "SCREW \nTERMINALS"
- note added: "SIGNAL CABLE\n26 CONDUCTOR RIBBON, 2x13 IDC CONN\nSee Note"
- note added: "Upper Deck Screw Terminals"
- note removed: "HEATER DRIVER OUTPUT MODULE\n0.2" PITCH SCREW TERMINALS"
- note removed: "RTD TEMPERATURE SENSOR MODULE\n0.2" PITCH SCREW TERMINALS"
- note removed: "SIGNAL CABLE\n26 CONDUCTOR RIBBON"
- moved on the sheet: DC-OUTPUT?, PS?, RTD-INPUT?
Changed lines of the file:
@@
 U 1 1 5955D4FC
 P 2650 2450
-F 0 "CONTROL?" H 2650 2550 60  0000 C CNN
+F 0 "CONTROL?" H 2650 2525 60  0000 C CNN
 F 1 "GTC01_CONTROLLER" H 2650 2350 60  0000 C CNN
 F 2 "" H 2350 2175 60  0001 C CNN
@@
 U 2 1 5955D5C0
 P 4600 2450
-F 0 "CONTROL?" H 4600 2550 60  0000 C CNN
+F 0 "CONTROL?" H 4600 2525 60  0000 C CNN
 F 1 "GTC01_CONTROLLER" H 4600 2350 60  0000 C CNN
 F 2 "" H 4300 2175 60  0001 C CNN
@@
 L GTC02_RTD_R1 RTD-INPUT?
 U 1 1 5955D756
-P 6900 2425
-F 0 "RTD-INPUT?" H 6900 2625 60  0000 C CNN
-F 1 "GTC02_RTD_R1" H 6900 2525 60  0000 C CNN
-F 2 "" H 6050 2375 60  0001 C CNN
-F 3 "" H 6050 2375 60  0001 C CNN
-F 4 "_" H 6900 2425 60  0001 C CNN "MPN"
-F 5 "_" H 6900 2425 60  0001 C CNN "HPN"
-F 6 "_" H 6900 2425 60  0001 C CNN "MFG"
-	1    6900 2425
+P 7300 2425
+F 0 "RTD-INPUT?" H 7300 2475 60  0000 C CNN
+F 1 "GTC02_RTD_R1" H 7300 2325 60  0000 C CNN
+F 2 "" H 6450 2375 60  0001 C CNN
+F 3 "" H 6450 2375 60  0001 C CNN
+F 4 "_" H 7300 2425 60  0001 C CNN "MPN"
+F 5 "_" H 7300 2425 60  0001 C CNN "HPN"
+F 6 "_" H 7300 2425 60  0001 C CNN "MFG"
+	1    7300 2425
 	1    0    0    -1
 $EndComp
@@
 L GTC03_HTR_R1 DC-OUTPUT?
 U 1 1 5955D810
-P 9525 2425
-F 0 "DC-OUTPUT?" H 9525 2575 60  0000 C CNN
-F 1 "GTC03_HTR_R1" H 9525 2475 60  0000 C CNN
-F 2 "" H 8675 2325 60  0001 C CNN
-F 3 "" H 8675 2325 60  0001 C CNN
-F 4 "_" H 9525 2425 60  0001 C CNN "MPN"
-F 5 "_" H 9525 2425 60  0001 C CNN "MFG"
-F 6 "_" H 9525 2425 60  0001 C CNN "HPN"
-	1    9525 2425
-	1    0    0    -1
-$EndComp
+P 9700 2425
+F 0 "DC-OUTPUT?" H 9700 2475 60  0000 C CNN
+F 1 "GTC03_HTR_R1" H 9700 2325 60  0000 C CNN
+F 2 "" H 8850 2325 60  0001 C CNN
+F 3 "" H 8850 2325 60  0001 C CNN
+F 4 "_" H 9700 2425 60  0001 C CNN "MPN"
+F 5 "_" H 9700 2425 60  0001 C CNN "MFG"
+F 6 "_" H 9700 2425 60  0001 C CNN "HPN"
+	1    9700 2425
+	1    0    0    -1
+$EndComp
+Text Label 7850 3375 3    60   ~ 0
+RTD1_F-
+Text Label 7750 3375 3    60   ~ 0
+RTD1_M-
+Text Label 7650 3375 3    60   ~ 0
+RTD1_M+
+Text Label 7550 3375 3    60   ~ 0
+RTD1_F+
 Text Label 7450 3375 3    60   ~ 0
-RTD1_F-
-Text Label 7350 3375 3    60   ~ 0
-RTD1_M-
-Text Label 7250 3375 3    60   ~ 0
-RTD1_M+
+H1_SHIELD
 Text Label 7150 3375 3    60   ~ 0
-RTD1_F+
+H2_SHIELD
+Text Label 6750 3375 3    60   ~ 0
+RTD2_F+
+Text Label 6850 3375 3    60   ~ 0
+RTD2_M+
+Text Label 6950 3375 3    60   ~ 0
+RTD2_M-
 Text Label 7050 3375 3    60   ~ 0
-H1_SHIELD
-Text Label 6750 3375 3    60   ~ 0
-H2_SHIELD
-Text Label 6350 3375 3    60   ~ 0
-RTD2_F+
-Text Label 6450 3375 3    60   ~ 0
-RTD2_M+
-Text Label 6550 3375 3    60   ~ 0
-RTD2_M-
-Text Label 6650 3375 3    60   ~ 0
 RTD2_F-
 Text Label 6300 6450 0    60   ~ 0
@@
 Text Label 6300 6550 0    60   ~ 0
 HEATER1+
-Text Label 9175 3375 3    60   ~ 0
+Text Label 9350 3375 3    60   ~ 0
 HEATER1-
-Text Label 8975 3375 3    60   ~ 0
+Text Label 9150 3375 3    60   ~ 0
 HEATER1+
-Text Label 9875 3375 3    60   ~ 0
+Text Label 10050 3375 3    60   ~ 0
 HEATER2-
-Text Label 10075 3375 3    60   ~ 0
+Text Label 10250 3375 3    60   ~ 0
 HEATER2+
 $Comp
@@
 L DC_Supply_48V PS?
 U 1 1 5956CD53
-P 9325 1225
-F 0 "PS?" H 9525 1475 60  0000 L CNN
-F 1 "DC_Supply_48V" H 9525 1375 60  0000 L CNN
-F 2 "No Footprint" H 9375 1975 50  0001 L CNN
-F 3 "No Datasheet" H 9375 1875 50  0001 L CNN
-F 4 "No HPN" H 9375 1575 50  0001 L CNN "HPN"
-F 5 "No MFG" H 9375 1775 50  0001 L CNN "MFG"
-F 6 "No MPN" H 9375 1675 50  0001 L CNN "MPN"
-	1    9325 1225
+P 9500 1225
+F 0 "PS?" H 9700 1475 60  0000 L CNN
+F 1 "DC_Supply_48V" H 9700 1375 60  0000 L CNN
+F 2 "No Footprint" H 9550 1975 50  0001 L CNN
+F 3 "No Datasheet" H 9550 1875 50  0001 L CNN
+F 4 "No HPN" H 9550 1575 50  0001 L CNN "HPN"
+F 5 "No MFG" H 9550 1775 50  0001 L CNN "MFG"
+F 6 "No MPN" H 9550 1675 50  0001 L CNN "MPN"
+	1    9500 1225
 	-1   0    0    -1
 $EndComp
@@
 Wire Wire Line
 	3125 5825 3525 5825
+Text Label 7850 1475 1    60   ~ 0
+X1-1
+Text Label 7750 1475 1    60   ~ 0
+X1-2
+Text Label 7650 1475 1    60   ~ 0
+X1-23
+Text Label 7550 1475 1    60   ~ 0
+X1-22
 Text Label 7450 1475 1    60   ~ 0
-X1-1
+X1-21
 Text Label 7350 1475 1    60   ~ 0
-X1-2
+X1-20
+Text Label 9950 3375 3    60   ~ 0
+X1-13
 Text Label 7250 1475 1    60   ~ 0
-X1-23
-Text Label 7150 1475 1    60   ~ 0
-X1-22
-Text Label 7050 1475 1    60   ~ 0
-X1-21
-Text Label 6950 1475 1    60   ~ 0
-X1-20
-Text Label 9775 3375 3    60   ~ 0
-X1-13
-Text Label 6850 1475 1    60   ~ 0
 X1-14
-NoConn ~ 6550 1475
-NoConn ~ 6450 1475
-NoConn ~ 6350 1475
+NoConn ~ 6950 1475
+NoConn ~ 6850 1475
+NoConn ~ 6750 1475
 $Comp
 L GTC01_CONTROLLER CONTROL?
@@
 NoConn ~ 4825 5725
 NoConn ~ 4825 5825
-Text Label 9475 3375 3    60   ~ 0
+Text Label 9650 3375 3    60   ~ 0
 X1-1
-Text Label 9575 3375 3    60   ~ 0
+Text Label 9750 3375 3    60   ~ 0
 X1-2
-Text Label 9375 3375 3    60   ~ 0
+Text Label 9550 3375 3    60   ~ 0
 X1-3
-Text Label 9675 3375 3    60   ~ 0
+Text Label 9850 3375 3    60   ~ 0
 X1-4
-Text Label 9275 3375 3    60   ~ 0
+Text Label 9450 3375 3    60   ~ 0
 X1-12
-Text Label 6750 1475 1    60   ~ 0
+Text Label 7150 1475 1    60   ~ 0
 X1-15
-Text Label 6650 1475 1    60   ~ 0
+Text Label 7050 1475 1    60   ~ 0
 X1-16
 $Comp
@@
 Wire Notes Line
 	5600 500  5600 7950
-Text Notes 775  900  0    60   ~ 0
+Text Notes 800  725  0    60   ~ 0
 CONTROLLER MODULE
 Wire Notes Line
@@
 Text Notes 7525 5475 0    60   ~ 0
 HEATER CONNECTION\nPHOENIX CONTACT PTSM PLUG, PN 1704858
-Text Notes 10125 775  2    60   ~ 0
-HEATER DRIVER OUTPUT MODULE\n0.2" PITCH SCREW TERMINALS
-Text Notes 7600 800  2    60   ~ 0
-RTD TEMPERATURE SENSOR MODULE\n0.2" PITCH SCREW TERMINALS
+Text Notes 10125 675  2    60   ~ 0
+HEATER DRIVER OUTPUT MODULE
+Text Notes 7600 700  2    60   ~ 0
+RTD TEMPERATURE SENSOR MODULE
 Wire Wire Line
 	3350 1450 3350 1000
@@
 L Earth #PWR?
 U 1 1 5958C6AB
-P 8725 1475
-F 0 "#PWR?" H 8725 1225 50  0001 C CNN
-F 1 "Earth" H 8725 1325 50  0001 C CNN
-F 2 "" H 8725 1475 50  0001 C CNN
-F 3 "" H 8725 1475 50  0001 C CNN
-	1    8725 1475
+P 8900 1475
+F 0 "#PWR?" H 8900 1225 50  0001 C CNN
+F 1 "Earth" H 8900 1325 50  0001 C CNN
+F 2 "" H 8900 1475 50  0001 C CNN
+F 3 "" H 8900 1475 50  0001 C CNN
+	1    8900 1475
 	1    0    0    -1
 $EndComp
@@
 L Earth #PWR?
 U 1 1 5958C8A3
-P 6850 4325
-F 0 "#PWR?" H 6850 4075 50  0001 C CNN
-F 1 "Earth" H 6850 4175 50  0001 C CNN
-F 2 "" H 6850 4325 50  0001 C CNN
-F 3 "" H 6850 4325 50  0001 C CNN
-	1    6850 4325
-	1    0    0    -1
-$EndComp
-Wire Wire Line
-	6850 4325 6850 3375
-NoConn ~ 6950 3375
-NoConn ~ 9075 3375
-NoConn ~ 9975 3375
-Wire Notes Line
-	6775 3375 6775 4275
-Wire Notes Line
-	6775 4275 6250 4275
-Wire Notes Line
-	6250 4275 6250 3400
-Text Notes 6325 4200 0    40   ~ 0
+P 7250 4325
+F 0 "#PWR?" H 7250 4075 50  0001 C CNN
+F 1 "Earth" H 7250 4175 50  0001 C CNN
+F 2 "" H 7250 4325 50  0001 C CNN
+F 3 "" H 7250 4325 50  0001 C CNN
+	1    7250 4325
+	1    0    0    -1
+$EndComp
+Wire Wire Line
+	7250 4325 7250 3375
+NoConn ~ 7350 3375
+NoConn ~ 9250 3375
+NoConn ~ 10150 3375
+Wire Notes Line
+	7175 3375 7175 4275
+Wire Notes Line
+	7175 4275 6650 4275
+Wire Notes Line
+	6650 4275 6650 3400
+Text Notes 6725 4200 0    40   ~ 0
 RTD2 CABLE\n20AWG/4\n+SHIELD
 Wire Notes Line
-	7475 4275 7475 3400
-Wire Notes Line
-	6975 4275 7475 4275
-Wire Notes Line
-	6975 4275 6975 3425
-Text Notes 7025 4200 0    40   ~ 0
+	7875 4275 7875 3400
+Wire Notes Line
+	7375 4275 7875 4275
+Wire Notes Line
+	7375 4275 7375 3425
+Text Notes 7425 4200 0    40   ~ 0
 RTD1 CABLE\n20AWG/4\n+SHIELD
 Wire Wire Line
-	8725 1475 9425 1475
-Wire Wire Line
-	9325 1225 9625 1225
-Wire Wire Line
-	9625 1225 9625 1475
-Wire Wire Line
-	9325 1325 9525 1325
-Wire Wire Line
-	9525 1325 9525 1475
-Wire Notes Line
-	10075 4275 10075 3400
-Wire Notes Line
-	8875 4275 10075 4275
-Wire Notes Line
-	9775 4275 9775 3400
-Wire Notes Line
-	9175 4275 9175 3400
-Wire Notes Line
-	8875 4275 8875 3400
-Text Notes 9200 4200 0    40   ~ 0
+	8900 1475 9600 1475
+Wire Wire Line
+	9500 1225 9800 1225
+Wire Wire Line
+	9800 1225 9800 1475
+Wire Wire Line
+	9500 1325 9700 1325
+Wire Wire Line
+	9700 1325 9700 1475
+Wire Notes Line
+	10350 4275 10350 3400
+Wire Notes Line
+	8950 4275 10350 4275
+Wire Notes Line
+	9950 4275 9950 3400
+Wire Notes Line
+	9350 4275 9350 3400
+Wire Notes Line
+	8950 4275 8950 3425
+Text Notes 9375 4100 0    40   ~ 0
 SIGNAL CABLE\n26 COND. RIBBON
 Wire Notes Line
-	7450 1450 7450 850
-Wire Notes Line
-	7450 850  6550 850
-Wire Notes Line
-	6550 850  6550 1425
-Text Notes 6725 1025 0    40   ~ 0
+	7850 1450 7850 850
+Wire Notes Line
+	7850 850  6950 850
+Wire Notes Line
+	6950 850  6950 1425
+Text Notes 7125 1025 0    40   ~ 0
 SIGNAL CABLE\n26 COND. RIBBON
-Text Notes 2250 6175 0    40   ~ 0
-SIGNAL CABLE\n26 CONDUCTOR RIBBON
-Text Notes 800  2450 0    60   ~ 0
-SCREW TERMINALS
-Text Notes 900  5075 0    60   ~ 0
+Text Notes 2100 6300 0    40   ~ 0
+SIGNAL CABLE\n26 CONDUCTOR RIBBON, 2x13 IDC CONN\nSee Note
+Text Notes 900  5075 0    50   ~ 0
 PCB HEADERS
 Text Label 4300 3700 2    60   ~ 0
@@
 Text Notes 875  4075 0    60   ~ 0
 COM PORTS
+Text Notes 1475 2525 0    60   ~ 0
+DIN\nRAIL
+Text Notes 5725 -300 0    60   ~ 0
+SCREW TERMINALS
+Text Notes 5800 1550 0    50   ~ 0
+SCREW TERMINALS
+Text Notes 5800 3350 0    50   ~ 0
+SCREW TERMINALS
+Text Notes 8250 3300 0    50   ~ 0
+SCREW TERMINALS
+Text Notes 9900 1625 0    50   ~ 0
+SCREW \nTERMINALS
+Wire Notes Line
+	10450 2600 1350 2600
+Wire Notes Line
+	1350 2600 1350 2325
+Wire Notes Line
+	1350 2325 10450 2325
+Wire Notes Line
+	10450 2325 10450 2600
+Text Notes 3975 2225 0    50   ~ 0
+Upper Deck Screw Terminals
+Text Notes 2250 2275 0    50   ~ 0
+Lower Deck Screw Terminals
+Wire Notes Line
+	1600 4575 1600 6350
+Wire Notes Line
+	1600 6350 3675 6350
+Wire Notes Line
+	3675 6350 3675 4575
+Text Notes 8975 4225 0    40   ~ 0
+HTR1 CABLE\n20AWG/2
+Text Notes 9975 4175 0    40   ~ 0
+HTR2 CABLE\n20AWG/2
 $EndSCHEMATC

Commit message: GTC_SYSTEM_01, REV 1
Parts:
- gave numbers to parts that had none: 7
Connections:
- net at CONTROL1.GND: now also PS1.2 (GND)
- net at CONTROL1.VIN (12-24VDC): now also PS1.1 (+24VDC)
- net X1-1 renamed 1_5V
- net X1-12 renamed 7_CTRL1
- net X1-13 renamed 12_CTRL2
- net X1-14 renamed 7_RDY1
- net X1-15 renamed 8_CS2
- net X1-16 renamed 9_RDY2
- net X1-2 renamed 10_GND
- net X1-20 renamed 6_CS1
- net X1-21 renamed 5_SDI
- net X1-22 renamed 4_SDO
- net X1-23 renamed 3_CLK
- net X1-3 renamed 8_ISENSE1
- net X1-4 renamed 11_ISENSE2
Other:
- note added: "26 COND. RIBBON\n26 AWG\n\nTO HEATER\nDRIVER MODULE\nSCREW TERMINALS\n\nSOUTH SIDE OF DIN"
- note added: "26 COND. RIBBON\n26 AWG\n\nTO RTD TEMP.\nSENSOR MODULE\nSCREW TERMINALS\n\nNORTH SIDE OF DIN"
- note added: "2X13 IDC\nPLUG CONN\n0.1" PITCH PINS\nAT CABLE CENTER\n\nConnect to \nX1 PCB Header\n2x13 Shrouded\nOn 'UPPER DECK'\nof Controller"
- note added: "DRIVER MODULE"
- note added: "HEATER CABLES\nPHOENIX CONTACT PTSM PLUG, PN 1704858"
- note added: "LOWER DECK"
- note added: "RTD MODULE"
- note added: "SCREW TERMINAL TERMINATION AT 2 ENDS\n2X13 IDC PLUG AT CENTER"
- note added: "UPPER DECK"
- note added: "UPPER DECK\nCOM PORTS"
- note added: "UPPER DECK\nPCB HEADERS"
- note added: "X1"
- note removed: "26 COND. RIBBON\n26 AWG\n\nTO HEATER\nDRIVER MODULE\nSCREW TERMINALS\n\nSOUTH SIDE"
- note removed: "26 COND. RIBBON\n26 AWG\n\nTO RTD TEMP.\nSENSOR MODULE\nSCREW TERMINALS\n\nNORTH SIDE"
- note removed: "2X13 IDC\nPLUG CONN\n0.1" PITCH PINS\nAT CABLE CENTER\n\nRECEPT. ON 'TOP'"
- note removed: "COM PORTS"
- note removed: "HEATER CONNECTION\nPHOENIX CONTACT PTSM PLUG, PN 1704858"
- note removed: "Lower Deck Screw Terminals"
- note removed: "PCB HEADERS"
- note removed: "SCREW \nTERMINALS"
- note removed: "Upper Deck Screw Terminals"
- moved on the sheet: DC-OUTPUT1, PS2, RTD-INPUT1

Commit message: GTC_STSTEM_01 Rev1, release
Connections:
- net X1-17 is gone; now on net 7_CTRL1: CONTROL1.X117 (D5)
- net X1-6 is gone; now on net 8_ISENSE1: CONTROL1.X106 (A3)
- net 12_CTRL2: now also CONTROL1.X115 (D3); no longer CONTROL1.X113 (D1)
- net 7_CTRL1: no longer CONTROL1.X112 (D0)
- net 8_CS2: now also CONTROL1.X116 (D4); no longer CONTROL1.X115 (D3)
- net 8_ISENSE1: no longer CONTROL1.X103 (A0)
- net at CONTROL1.GND: now also PS1.2 (GND)
- net at CONTROL1.VIN (12-24VDC): now also PS1.1 (+24VDC)
- net 10_CS3: now reaches RTD-INPUT1.10 (CS3)
- net 10_CS3: now also CONTROL1.X114 (D2)
- net 11_CS4: now reaches RTD-INPUT1.11 (CS4)
- net 11_CS4: now also CONTROL1.X112 (D0)
- net 7_RDY1: no longer names the net of RTD-INPUT1.7 (RDY1)
- net 7_RDY1: no longer CONTROL1.X114 (D2)
- net 9_RDY2: no longer names the net of RTD-INPUT1.9 (RDY2)
- net 9_RDY2: no longer CONTROL1.X116 (D4)
- new net X1-13: CONTROL1.X113 (D1)
- new net X1-3: CONTROL1.X103 (A0)
Other:
- note added: "24V Logic\nActive High"
- note added: "RS485 Cable\n22AWG/4\n+SHIELD"
Changed lines of the file:
@@
 X1-20
 Text Label 9600 3375 3    60   ~ 0
-X1-13
-Text Label 6900 1475 1    60   ~ 0
-X1-14
-NoConn ~ 6600 1475
-NoConn ~ 6500 1475
+X1-15
 NoConn ~ 6400 1475
 $Comp
@@
 X1-2
 Text Label 9200 3375 3    60   ~ 0
-X1-3
+X1-6
 Text Label 9500 3375 3    60   ~ 0
 X1-4
 Text Label 9100 3375 3    60   ~ 0
+X1-17
+Text Label 6500 1475 1    60   ~ 0
 X1-12
-Text Label 6800 1475 1    60   ~ 0
-X1-15
-Text Label 6700 1475 1    60   ~ 0
-X1-16
 $Comp
 L GTC01_CONTROLLER CONTROL1
 U 5 1 59585CEB
 P 2275 3800
-F 0 "CONTROL1" H 2275 3900 60  0000 C CNN
-F 1 "GTC01_CONTROLLER" H 2275 3700 60  0000 C CNN
+F 0 "CONTROL1" H 2250 3700 60  0000 C CNN
+F 1 "GTC01_CONTROLLER" H 2250 3400 60  0000 C CNN
 F 2 "" H 1975 3525 60  0001 C CNN
 F 3 "" H 1975 3525 60  0001 C CNN
@@
 Text Notes 6650 2200 0    50   ~ 0
 SCREW TERMINALS
-Text Notes 3975 2225 0    50   ~ 0
+Text Notes 3975 2250 0    50   ~ 0
 UPPER DECK
 Text Notes 3000 2250 0    50   ~ 0
@@
 SCREW TERMINALS
 Text Label 4450 7600 0    60   ~ 0
-X1-13
+X1-15
 Text Label 4450 7300 0    60   ~ 0
 X1-1
@@
 X1-2
 Text Label 4450 7200 0    60   ~ 0
-X1-3
+X1-6
 Text Label 4450 7500 0    60   ~ 0
 X1-4
 Text Label 4450 7100 0    60   ~ 0
-X1-12
+X1-17
 Text Label 1450 6900 2    60   ~ 0
 X1-1
@@
 X1-20
 Text Label 1450 7500 2    60   ~ 0
-X1-14
-Text Label 1450 7600 2    60   ~ 0
-X1-15
+X1-16
 Text Label 1450 7700 2    60   ~ 0
-X1-16
+X1-12
 Text Notes 2800 6800 0    60   ~ 0
 X1
@@
 Text Label 650  7400 0    60   ~ 0
 6_CS1
-Text Label 650  7500 0    60   ~ 0
-7_RDY1
 Text Label 650  7600 0    60   ~ 0
-8_CS2
-Text Label 650  7700 0    60   ~ 0
-9_RDY2
+10_CS3
 Text Label 5000 7100 0    60   ~ 0
 7_CTRL1
@@
 12_CTRL2
 Wire Wire Line
-	6300 5850 7100 5850
+	6300 5850 6950 5850
+Wire Wire Line
+	6950 5850 7100 5850
 Wire Wire Line
 	6300 5750 6850 5750
@@
 	6850 6050 6950 5950
 Wire Wire Line
-	6300 5950 7100 5950
+	6300 5950 6950 5950
+Wire Wire Line
+	6950 5950 7100 5950
 Connection ~ 6950 5950
 Connection ~ 6950 5850
@@
 	6950 6050 7100 6050
 Wire Wire Line
-	8650 5850 9450 5850
+	8650 5850 9300 5850
+Wire Wire Line
+	9300 5850 9450 5850
 Wire Wire Line
 	8650 5750 9200 5750
@@
 	9200 6050 9300 5950
 Wire Wire Line
-	8650 5950 9450 5950
+	8650 5950 9300 5950
+Wire Wire Line
+	9300 5950 9450 5950
 Connection ~ 9300 5950
 Connection ~ 9300 5850
@@
 	8600 4300 8600 3450
 Wire Notes Line
-	7500 1450 7500 850
-Wire Notes Line
-	7500 850  6600 850
-Wire Notes Line
-	6600 850  6600 1425
+	7525 1450 7525 850
+Wire Notes Line
+	7525 850  6325 850
+Wire Notes Line
+	6325 850  6325 1475
 Wire Wire Line
 	5100 3450 5100 3700
@@
 	650  7400 1450 7400
 Wire Wire Line
-	650  7500 1450 7500
-Wire Wire Line
 	650  7600 1450 7600
-Wire Wire Line
-	650  7700 1450 7700
 Wire Notes Line
 	550  6750 1000 6750
@@
 Text Notes 900  2050 0    50   ~ 0
 SCREW TERMINALS
+NoConn ~ 6700 1475
+NoConn ~ 6900 1475
+Text Label 6800 1475 1    60   ~ 0
+X1-16
+Text Label 6600 1475 1    60   ~ 0
+X1-14
+Text Notes 4175 800  0    60   ~ 0
+24V Logic\nActive High
+$Comp
+L Earth #PWR?
+U 1 1 5956EE24
+P 5400 4225
+F 0 "#PWR?" H 5400 3975 50  0001 C CNN
+F 1 "Earth" H 5400 4075 50  0001 C CNN
+F 2 "" H 5400 4225 50  0001 C CNN
+F 3 "" H 5400 4225 50  0001 C CNN
+	1    5400 4225
+	1    0    0    -1
+$EndComp
+Text Label 4300 4100 2    60   ~ 0
+RS485_Cable_Shield
+Wire Wire Line
+	4300 4100 5400 4100
+Wire Wire Line
+	5400 4100 5400 4225
+Wire Notes Line
+	4775 3550 3100 3550
+Wire Notes Line
+	3100 3550 3100 4150
+Wire Notes Line
+	3100 4150 4825 4150
+Text Notes 3600 3875 2    50   ~ 0
+RS485 Cable\n22AWG/4\n+SHIELD
+Text Label 1450 7600 2    60   ~ 0
+X1-14
+Text Label 650  7700 0    60   ~ 0
+11_CS4
+Wire Wire Line
+	650  7700 1450 7700
+Text Label 650  7500 0    60   ~ 0
+8_CS2
+Wire Wire Line
+	650  7500 1450 7500
 $EndSCHEMATC

Commit message: Revision 2
Parts:
- removed PS1: DC_Supply_24V, No Footprint, symbol DC_Supply_24V
- added PLUG3: RTA_GATEWAY_PORT_0, No Footprint, symbol RTA_GATEWAY_PORT_0
- added PS3: DC_Supply_12V, No Footprint, symbol DC_Supply_12V
- added PS?: DC_Supply_24V, No Footprint, symbol DC_Supply_24V
Connections:
- net 10_CS3: no longer RTD-INPUT1.10 (CS3)
- net 10_GND: no longer DC-OUTPUT1.10 (GND), RTD-INPUT1.2 (GND)
- net 11_CS4: no longer RTD-INPUT1.11 (CS4)
- net 11_ISENSE2: no longer DC-OUTPUT1.11 (ISENSE2)
- net 12_CTRL2: no longer DC-OUTPUT1.12 (CTRL2)
- net 1_5V: no longer DC-OUTPUT1.9 (5V), RTD-INPUT1.1 (5V)
- net 3_CLK: no longer RTD-INPUT1.3 (CLK)
- net 4_SDO: no longer RTD-INPUT1.4 (SDO)
- net 5_SDI: no longer RTD-INPUT1.5 (SDI)
- net 6_CS1: no longer RTD-INPUT1.6 (CS1)
- net 7_CTRL1: no longer DC-OUTPUT1.7 (CTRL1)
- net 8_CS2: no longer RTD-INPUT1.8 (CS2)
- net 8_ISENSE1: no longer DC-OUTPUT1.8 (ISENSE1)
- net ALARM_1: now also CONTROL1.R0B (Relay0B_d22); no longer CONTROL1.D10 (D10_d12)
- net ALARM_2: now also CONTROL1.R1B (Relay1B_d23); no longer CONTROL1.D11 (D11_d13)
- net Earth: now also PLUG3.4 (PE)
- net RS485_A: now also PLUG3.3 (TX+); no longer CONTROL1.+ (RS485_A)
- net RS485_B: now also PLUG3.2 (TX-); no longer CONTROL1.- (RS485_B)
- net at CONTROL1.GND: now also PS3.2 (GND)
- net +24V: now reaches CONTROL1.R0A (Relay0A_d22)
- net +24V: now also CONTROL1.R1A (Relay1A_d23), PS?.1 (+24VDC)
- net at CONTROL1.VIN (12-24VDC): now also PS3.1 (+12VDC)
- net RS485_5V: no longer names the net of CONTROL1.+5V
- removed net RS485_GND: CONTROL1.GND
- new net 24V: PLUG3.5 (PWRIN)
- new net GND: PLUG3.1 (GND), PS?.2 (GND)
- new net RS485-A: CONTROL1.+ (RS485_A)
- new net RS485-B: CONTROL1.- (RS485_B)
- no-connect marks 81 -> 96
Other:
- note added: "22AWG/2 Twisted Pair + Shield"
- note added: "26 cond\nribbon cable"
- note added: "2x13 Signal \nHeader"
- note added: "CONTROLLER"
- note added: "CONTROLLER MODULE\nX1 Header"
- note added: "Cable Shield\nEarth/Chassis"
- note added: "DRIVER MODULE\nSignal Header"
- note added: "RS485 Cable"
- note added: "RTA GATEWAY"
- note added: "RTD MODULE\nSignal Header"
- note added: "SCREW\nTERMINALS"
- note added: "SIGNAL CABLE\nReference"
- note added: "Signal Cable Reference"
- note added: "Signal Cable\n26 Conductor Ribbon\n3x, 26pin Sockets on Cable\nCable ships with Modules\n\nPanel Builder Terminate Sockets \nto Signal Headers on Modules"
- note added: "X1 HEADER"
- note added: "X2 HEADER"
- note removed: "24V Logic\nActive High"
- note removed: "DRIVER MODULE"
- note removed: "RS485 Cable\n22AWG/4\n+SHIELD"
- note removed: "RTD MODULE"
- note removed: "SIGNAL CABLE\n26 COND. RIBBON"
- note removed: "SIGNAL CABLE\n26 CONDUCTOR RIBBON, 2x13 IDC CONN\nSee Note"
- moved on the sheet: CONTROL1C, CONTROL1D, CONTROL1E, PLUG1, PLUG2
